File: epaper_eval/WFT0420CZ15_eval.sch (EAGLE design)
At the start: 15 parts, among them CN1 WFT0420CZ15_IF, CN2 WFT0420CZ15

Commit message: 部品を追加
Parts:
- added C10, C12: 1uF50V, Parts:CAP_0805
- added C11: 4.7uF50V, Parts:CAP_0805
- added C13: 0.1uF, Parts:CAP_0805
- added D1, D2, D3: MBR0530, Parts:MBR0530
- added L1: 10uH, Parts:NLCV25T
- added Q1: SI1308EDL, Parts:SI1308EDL
- added R1: 0.47, Parts:RESISTOR_0805
- added R2, R3: 4.7k, Parts:RESISTOR_0805
- added U1: LM75BIMM-3, Parts:LM75BIMM-3
- C9: device Parts:TPST106K016R0800 -> Parts:CAP_0805
Connections:
- new net GDR: CN2.GDR, Q1.G
- new net N$15: C11.2, D2.A, D3.C
- new net N$6: C11.1, D1.A, L1.2, Q1.D
- new net PREVGH: C10.1, CN2.PREVGH, D1.C
- new net PREVGL: C12.1, CN2.PREVGL, D3.A
- new net RESE: CN2.RESE, Q1.S, R1.2
- new net TSCL: CN2.TSCL, R3.1, U1.SCL
- new net TSDA: CN2.TSDA, R2.1, U1.SDA
- net +3V3: now also C13.1, C9.1, L1.1, R2.2, R3.2, U1.+VS; no longer C9.+
- net 0V: now also C10.2, C12.2, C13.2, C9.2, D2.C, R1.1, U1.A0, U1.A1, U1.A2, U1.GND; no longer C9.-
Other:
- moved on the sheet: H1, H2, H3, H4

Commit message: レイアウト変更
概ね確定です
Parts:
- added C14: 10uF16V, Parts:TPST106K016R0800
- added R4: 100k, Parts:RESISTOR_0805
Connections:
- net +3V3: now also C14.+
- net 0V: now also C14.-, R4.1
- net GDR: now also R4.2
Changed lines of the file:
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@@
 <part name="GND4" library="Supply" deviceset="0V" device=""/>
 <part name="C13" library="Parts" deviceset="CAP" device="_0805" value="0.1uF"/>
+<part name="R4" library="Parts" deviceset="RESISTOR" device="_0805" value="100k"/>
+<part name="C14" library="Parts" deviceset="TPST*" device="106K016R0800" value="10uF16V"/>
 </parts>
 <sheets>
@@
 <instance part="GND4" gate="1" x="231.14" y="35.56"/>
 <instance part="C13" gate="G$1" x="236.22" y="55.88"/>
+<instance part="R4" gate="G$1" x="66.04" y="38.1" rot="R90"/>
+<instance part="C14" gate="G$1" x="33.02" y="55.88"/>
 </instances>
 <busses>
@@
 <wire x1="48.26" y1="127" x2="86.36" y2="127" width="0.1524" layer="91"/>
 <junction x="48.26" y="127"/>
+<pinref part="C14" gate="G$1" pin="+"/>
+<wire x1="33.02" y1="55.88" x2="33.02" y2="71.12" width="0.1524" layer="91"/>
+<wire x1="33.02" y1="71.12" x2="48.26" y2="71.12" width="0.1524" layer="91"/>
 </segment>
 <segment>
@@
 <pinref part="C9" gate="G$1" pin="2"/>
 <wire x1="48.26" y1="48.26" x2="48.26" y2="33.02" width="0.1524" layer="91"/>
-<wire x1="48.26" y1="33.02" x2="76.2" y2="33.02" width="0.1524" layer="91"/>
+<wire x1="48.26" y1="33.02" x2="66.04" y2="33.02" width="0.1524" layer="91"/>
+<pinref part="R4" gate="G$1" pin="1"/>
+<wire x1="66.04" y1="33.02" x2="76.2" y2="33.02" width="0.1524" layer="91"/>
+<wire x1="66.04" y1="38.1" x2="66.04" y2="33.02" width="0.1524" layer="91"/>
+<junction x="66.04" y="33.02"/>
+<pinref part="C14" gate="G$1" pin="-"/>
+<wire x1="33.02" y1="48.26" x2="33.02" y2="33.02" width="0.1524" layer="91"/>
+<wire x1="33.02" y1="33.02" x2="48.26" y2="33.02" width="0.1524" layer="91"/>
+<junction x="48.26" y="33.02"/>
 </segment>
 <segment>
@@
 <segment>
 <pinref part="Q1" gate="G$1" pin="G"/>
-<wire x1="71.12" y1="58.42" x2="55.88" y2="58.42" width="0.1524" layer="91"/>
+<wire x1="71.12" y1="58.42" x2="66.04" y2="58.42" width="0.1524" layer="91"/>
 <label x="55.88" y="58.42" size="1.778" layer="95"/>
-</segment>
-</net>
+<pinref part="R4" gate="G$1" pin="2"/>
+<wire x1="66.04" y1="58.42" x2="55.88" y2="58.42" width="0.1524" layer="91"/>
+<wire x1="66.04" y1="48.26" x2="66.04" y2="58.42" width="0.1524" layer="91"/>
+<junction x="66.04" y="58.42"/>
+</segment>
+</net>
