File: epaper_eval/WFT0420CZ15_conv.brd (EAGLE design)
At the start: 45 x 25 mm, 26 parts, among them CN1 WFT0420CZ15_IF, CN2 WFT0420CZ15-SMD_, Q1 PMF370XN_, U1 LM75BIMM-3_

Commit message: 部品配置を修正
Parts:
- moved C8 4.26 mm to (39.4, 1.91), turned to 180 degrees
- moved C2 3.19 mm to (39.4, 23.2)
- moved R2 2.54 mm to (26.7, 19.7)
- moved R3 2.22 mm to (20.0, 19.7)
- moved C1 2.01 mm to (34.3, 21.6), turned to 90 degrees
- moved C6 1.27 mm to (26.7, 3.81)
- moved D1 1.27 mm to (20.5, 4.45)
- moved C10 1.27 mm to (29.2, 3.81)
- moved C11 1.27 mm to (17.3, 4.45)
- moved C5 1.27 mm to (24.1, 3.81)
- moved C7 1.27 mm to (31.8, 3.81)
- moved C12 1.27 mm to (34.3, 3.81)
Routing:
- net +3V3: track 105.1 -> 114.3 mm
- net TSCL: track 18.8 -> 27.5 mm
- net 0V: track 49.9 -> 55.2 mm
- net TSDA: track 11.4 -> 16.0 mm
- net N$8: track 6.56 -> 10.0 mm
- net N$1: track 3.46 -> 6.71 mm
- net N$7: track 10.6 -> 8.62 mm
- net PREVGH: track 22.3 -> 20.7 mm
- net N$2: track 9.78 -> 8.23 mm
- net N$3: track 15.5 -> 14.2 mm
- net N$4: track 17.2 -> 15.9 mm
- net N$6: track 22.3 -> 22.8 mm
- net N$15: track 7.79 -> 7.27 mm

Commit message: 部品配置の小修正
Parts:
- moved L1 1.27 mm to (13.5, 9.68)
Routing:
- net N$9: track 38.8 -> 37.4 mm
- net +3V3: track 114.3 -> 115.5 mm
Changed lines of the file:
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@@
 <?xml version="1.0" encoding="utf-8"?>
 <!DOCTYPE eagle SYSTEM "eagle.dtd">
-<eagle version="7.7.0">
+<eagle version="7.5.0">
 <drawing>
 <settings>
@@
 <attribute name="VALUE" x="19.685" y="8.09625" size="0.7112" layer="27"/>
 </element>
-<element name="L1" library="Parts" package="NLCV25T" value="10uH" x="13.49375" y="8.41375"/>
+<element name="L1" library="Parts" package="NLCV25T" value="10uH" x="13.49375" y="9.68375"/>
 <element name="Q1" library="Parts" package="SOT323_DEV" value="PMF370XN_" x="11.43" y="18.25625" smashed="yes" rot="R270">
 <attribute name="NAME" x="10.00125" y="15.24" size="0.8128" layer="25" rot="R90"/>
@@
 <wire x1="1.11125" y1="6.985" x2="1.74625" y2="6.35" width="0.3048" layer="1"/>
 <wire x1="1.74625" y1="6.35" x2="3.81" y2="6.35" width="0.3048" layer="1"/>
-<wire x1="12.065" y1="5.745" x2="12.065" y2="8.335" width="0.6096" layer="1"/>
-<wire x1="12.065" y1="8.335" x2="12.14375" y2="8.41375" width="0.3048" layer="1"/>
 <wire x1="12.065" y1="5.745" x2="8.455" y2="5.745" width="0.6096" layer="1"/>
 <wire x1="8.455" y1="5.745" x2="8.255" y2="5.945" width="0.3048" layer="1"/>
@@
 <wire x1="18.7325" y1="20.47875" x2="18.7325" y2="19.715" width="0.3048" layer="1"/>
 <wire x1="18.7325" y1="19.715" x2="18.7025" y2="19.685" width="0.3048" layer="1"/>
+<wire x1="12.065" y1="5.745" x2="12.065" y2="9.605" width="0.6096" layer="1"/>
+<wire x1="12.065" y1="9.605" x2="12.14375" y2="9.68375" width="0.6096" layer="1"/>
 </signal>
 <signal name="N$7">
@@
 <contactref element="CN2" pad="9"/>
 <wire x1="38.26" y1="14.45" x2="35.715" y2="14.45" width="0.3048" layer="1"/>
-<wire x1="8.73125" y1="16.8275" x2="7.77875" y2="17.78" width="0.3048" layer="1"/>
-<wire x1="7.77875" y1="17.78" x2="7.77875" y2="20.16125" width="0.3048" layer="1"/>
-<wire x1="7.77875" y1="20.16125" x2="6.35" y2="21.59" width="0.3048" layer="1"/>
-<wire x1="6.35" y1="21.59" x2="3.81" y2="21.59" width="0.3048" layer="1"/>
 <wire x1="35.715" y1="14.45" x2="33.3375" y2="16.8275" width="0.3048" layer="1"/>
 <wire x1="33.3375" y1="16.8275" x2="8.73125" y2="16.8275" width="0.3048" layer="1"/>
+<wire x1="3.81" y1="21.59" x2="3.96875" y2="21.59" width="0.3048" layer="1"/>
+<wire x1="3.96875" y1="21.59" x2="8.73125" y2="16.8275" width="0.3048" layer="1"/>
 </signal>
 <signal name="N$10">
@@
 <contactref element="C11" pad="1"/>
 <via x="15.08125" y="18.25625" extent="1-16" drill="0.6"/>
-<wire x1="16.03375" y1="17.30375" x2="16.03375" y2="10.31875" width="0.4064" layer="16"/>
-<via x="16.03375" y="10.31875" extent="1-16" drill="0.6"/>
-<wire x1="16.03375" y1="10.31875" x2="16.03375" y2="9.60375" width="0.4064" layer="1"/>
-<wire x1="16.03375" y1="9.60375" x2="14.84375" y2="8.41375" width="0.4064" layer="1"/>
+<wire x1="16.03375" y1="17.30375" x2="16.03375" y2="12.3825" width="0.4064" layer="16"/>
+<via x="16.03375" y="12.3825" extent="1-16" drill="0.6"/>
+<wire x1="16.03375" y1="12.3825" x2="16.03375" y2="11.50875" width="0.4064" layer="1"/>
 <wire x1="12.83" y1="18.25625" x2="15.08125" y2="18.25625" width="0.4064" layer="1"/>
 <wire x1="16.03375" y1="17.30375" x2="15.08125" y2="18.25625" width="0.4064" layer="16"/>
-<wire x1="14.84375" y1="8.41375" x2="14.84375" y2="5.605" width="0.4064" layer="1"/>
+<wire x1="14.84375" y1="9.68375" x2="14.84375" y2="5.605" width="0.4064" layer="1"/>
 <wire x1="14.84375" y1="5.605" x2="17.30375" y2="3.145" width="0.4064" layer="1"/>
 <wire x1="17.30375" y1="3.145" x2="17.4925" y2="3.145" width="0.4064" layer="1"/>
@@
 <wire x1="18.25625" y1="2.38125" x2="20.4075" y2="2.38125" width="0.4064" layer="1"/>
 <wire x1="20.4075" y1="2.38125" x2="20.47875" y2="2.31" width="0.4064" layer="1"/>
+<wire x1="14.84375" y1="9.68375" x2="14.84375" y2="10.31875" width="0.4064" layer="1"/>
+<wire x1="14.84375" y1="10.31875" x2="16.03375" y2="11.50875" width="0.4064" layer="1"/>
 </signal>
 <signal name="GDR">
