File: epaper_eval/WFT0750CZ09_conv.brd (EAGLE design)
At the start: 45 x 28 mm, 26 parts, among them CN1 WFT0750CZ09_IF, CN2 WFT0750CZ09-SMD_, Q1 PMF370XN_, U1 LM75BIMM-3_

Commit message: 基板デザイン修正
Parts:
- moved D1 2.38 mm to (21.0, 2.54), turned to 180 degrees
- moved C11 2.16 mm to (21.0, 5.71), turned to 0 degrees
- moved L1 1.42 mm to (13.3, 10.2), turned to 180 degrees
- moved U1 1.42 mm to (27.9, 23.5), turned to 0 degrees
- moved C3 1.27 mm to (29.2, 10.5)
Routing:
- net 0V: track 51.3 -> 61.0 mm
- net TSCL: track 28.0 -> 20.8 mm
- net FCSB: track 37.3 -> 42.6 mm, vias 1 -> 2
- net PREVGH: track 18.9 -> 22.1 mm
- net +3V3: track 95.0 -> 97.7 mm
- net N$6: track 23.9 -> 26.0 mm
- net N$15: track 6.48 -> 8.28 mm
- net TSDA: track 23.2 -> 21.8 mm
- net N$5: track 6.70 -> 7.97 mm
- net FDSO: track 44.1 -> 43.0 mm
- net PREVGL: track 18.8 -> 18.1 mm

Commit message: 基板デザイン修正
Parts:
- moved C8 2.93 mm to (14.0, 7.30), turned to 0 degrees
- moved C9 1.93 mm to (14.0, 4.13), turned to 0 degrees
- moved C1 1.27 mm to (36.2, 22.9)
- moved C2 1.27 mm to (36.2, 25.4)
- moved C7 0.64 mm to (8.26, 3.81)
- moved L1 0.63 mm to (14.0, 10.2), turned to 0 degrees
Routing:
- net N$6: track 26.0 -> 21.4 mm
- net 0V: track 61.0 -> 59.4 mm
- net N$8: track 7.74 -> 8.52 mm
- net N$7: track 11.3 -> 12.1 mm

Commit message: 基板デザイン修正
Parts:
- C7: device Parts:C1210_TPST -> Parts:C1210_TPST_DEV
- L1: device Parts:NLCV25T -> Parts:NLCV25T_DEV
- moved C7 1.27 mm to (8.26, 5.08)
Routing:
- net +3V3: track 97.4 -> 91.0 mm
Changed lines of the file:
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@@
 <layer number="49" name="Reference" color="7" fill="1" visible="no" active="yes"/>
 <layer number="50" name="dxf" color="7" fill="1" visible="no" active="no"/>
-<layer number="51" name="tDocu" color="7" fill="1" visible="no" active="yes"/>
-<layer number="52" name="bDocu" color="7" fill="1" visible="no" active="yes"/>
+<layer number="51" name="tDocu" color="7" fill="1" visible="yes" active="yes"/>
+<layer number="52" name="bDocu" color="7" fill="1" visible="yes" active="yes"/>
 <layer number="53" name="tGND_GNDA" color="7" fill="9" visible="no" active="no"/>
 <layer number="54" name="bGND_GNDA" color="1" fill="9" visible="no" active="no"/>
@@
 <attribute name="VALUE" x="22.5425" y="26.9875" size="0.6096" layer="27" rot="R180"/>
 </element>
-<element name="C7" library="Parts" package="C1210_TPST" value="10uF16V" x="8.255" y="3.81" smashed="yes" rot="R270">
-<attribute name="NAME" x="8.89" y="8.5725" size="0.8128" layer="25" rot="R270"/>
-<attribute name="VALUE" x="5.3975" y="5.715" size="0.8128" layer="27" rot="R270"/>
+<element name="C7" library="Parts" package="C1210_TPST_DEV" value="10uF16V" x="8.255" y="5.08" smashed="yes" rot="R270">
+<attribute name="NAME" x="8.89" y="9.8425" size="0.8128" layer="25" rot="R270"/>
+<attribute name="VALUE" x="5.3975" y="6.985" size="0.8128" layer="27" rot="R270"/>
 </element>
 <element name="C2" library="Parts" package="SMD_2012" value="10uF50V" x="36.195" y="25.4" smashed="yes" rot="R180">
@@
 <attribute name="VALUE" x="19.685" y="6.985" size="0.7112" layer="27"/>
 </element>
-<element name="L1" library="Parts" package="NLCV25T" value="10uH" x="13.97" y="10.16"/>
+<element name="L1" library="Parts" package="NLCV25T_DEV" value="10uH" x="13.97" y="10.16"/>
 <element name="Q1" library="Parts" package="SOT323_DEV" value="PMF370XN_" x="11.43" y="18.25625" smashed="yes" rot="R270">
 <attribute name="NAME" x="10.00125" y="15.24" size="0.8128" layer="25" rot="R90"/>
@@
 <wire x1="12.67" y1="7.3025" x2="12.67" y2="4.1275" width="0.4572" layer="1"/>
 <wire x1="12.67" y1="7.3025" x2="12.67" y2="10.11" width="0.4572" layer="1"/>
-<wire x1="12.67" y1="10.11" x2="12.62" y2="10.16" width="0.4572" layer="1"/>
-<wire x1="3.81" y1="5.08" x2="8.025" y2="5.08" width="0.4572" layer="1"/>
-<wire x1="8.025" y1="5.08" x2="8.255" y2="5.31" width="0.4572" layer="1"/>
+<wire x1="12.67" y1="10.11" x2="12.42" y2="10.16" width="0.4572" layer="1"/>
 <wire x1="12.67" y1="4.1275" x2="11.1125" y2="4.1275" width="0.4572" layer="1"/>
-<wire x1="11.1125" y1="4.1275" x2="10.16" y2="5.08" width="0.4572" layer="1"/>
-<wire x1="10.16" y1="5.08" x2="8.485" y2="5.08" width="0.4572" layer="1"/>
-<wire x1="8.485" y1="5.08" x2="8.255" y2="5.31" width="0.4572" layer="1"/>
 <wire x1="27.91" y1="13.0175" x2="27.305" y2="13.0175" width="0.4064" layer="1"/>
 <wire x1="27.305" y1="13.0175" x2="26.9875" y2="13.335" width="0.4064" layer="1"/>
-<wire x1="26.9875" y1="13.335" x2="13.0175" y2="13.335" width="0.4064" layer="1"/>
-<wire x1="13.0175" y1="13.335" x2="8.255" y2="8.5725" width="0.4064" layer="1"/>
-<wire x1="8.255" y1="8.5725" x2="8.255" y2="5.31" width="0.4064" layer="1"/>
+<wire x1="26.9875" y1="13.335" x2="14.9225" y2="13.335" width="0.4064" layer="1"/>
+<wire x1="11.1125" y1="4.1275" x2="8.89" y2="6.35" width="0.4572" layer="1"/>
+<wire x1="8.89" y1="6.35" x2="8.685" y2="6.35" width="0.4572" layer="1"/>
+<wire x1="8.685" y1="6.35" x2="8.255" y2="6.78" width="0.4572" layer="1"/>
+<wire x1="12.67" y1="10.11" x2="12.67" y2="11.0825" width="0.4064" layer="1"/>
+<wire x1="12.67" y1="11.0825" x2="14.9225" y2="13.335" width="0.4064" layer="1"/>
+<wire x1="3.81" y1="5.08" x2="5.3975" y2="5.08" width="0.4572" layer="1"/>
+<wire x1="5.3975" y1="5.08" x2="6.985" y2="6.6675" width="0.4572" layer="1"/>
+<wire x1="6.985" y1="6.6675" x2="8.1425" y2="6.6675" width="0.4572" layer="1"/>
+<wire x1="8.1425" y1="6.6675" x2="8.255" y2="6.78" width="0.4572" layer="1"/>
 </signal>
 <signal name="N$7">
@@
 <wire x1="15.39875" y1="18.25625" x2="16.51" y2="17.145" width="0.4572" layer="16"/>
 <wire x1="15.32" y1="10.05" x2="19.655" y2="5.715" width="0.4572" layer="1"/>
-<wire x1="15.32" y1="10.16" x2="15.32" y2="10.05" width="0.4572" layer="1"/>
+<wire x1="15.52" y1="10.16" x2="15.32" y2="10.05" width="0.4572" layer="1"/>
 <wire x1="15.24" y1="12.065" x2="15.24" y2="10.24" width="0.4572" layer="1"/>
-<wire x1="15.24" y1="10.24" x2="15.32" y2="10.16" width="0.4572" layer="1"/>
+<wire x1="15.24" y1="10.24" x2="15.52" y2="10.16" width="0.4572" layer="1"/>
 <wire x1="16.51" y1="17.145" x2="16.51" y2="13.335" width="0.4572" layer="16"/>
 <wire x1="16.51" y1="13.335" x2="15.24" y2="12.065" width="0.4572" layer="16"/>

Commit message: 部品変更
Parts:
- removed R1: 10, Parts:SMD_2012
- added C14: 0.1uF50V, Parts:SMD_2012
- C10: value 10uF50V -> 0.1uF16V
- C11: value 4.7uF50V -> 10uF50V
- C12: value 10uF50V -> 4.7uF50V
- C13: value 0.1uF50V -> 10uF50V
- C4: value 10uF50V -> 1uF50V
- C6: value 1uF50V -> 10uF50V
- C7: value 10uF16V -> 1uF50V; device Parts:C1210_TPST_DEV -> Parts:SMD_2012
- C8: value 1uF16V -> 10uF16V; device Parts:SMD_2012 -> Parts:C1210_TPST_DEV
- C9: value 0.1uF16V -> 1uF16V
- moved C7 31.3 mm to (39.4, 1.91), turned to 180 degrees
- moved C13 25.7 mm to (34.3, 3.81), turned to 270 degrees
- moved C10 15.4 mm to (14.0, 5.71), turned to 0 degrees
- moved C12 13.5 mm to (21.0, 5.71), turned to 0 degrees
- moved C11 8.47 mm to (29.2, 3.81), turned to 270 degrees
- moved C6 7.85 mm to (31.8, 3.81), turned to 270 degrees
- moved C4 7.13 mm to (29.2, 10.5), turned to 180 degrees
- moved C8 5.54 mm to (8.89, 5.08), turned to 270 degrees
- moved C5 5.08 mm to (26.7, 3.81)
- moved C3 2.22 mm to (29.2, 12.7)
- moved C9 1.59 mm to (14.0, 2.54)
Connections:
- removed net N$4: CN2.15, CN2.16, R1.2
- net +3V3: now also C10.1, C14.1, C3.1, CN2.15, CN2.16; no longer C13.1, C7.1, R1.1
- net 0V: now also C11.2, C14.2; no longer C12.2
- net N$1: now also C7.1; no longer C6.1
- net N$15: now also C12.2; no longer C11.2
- net N$2: now also C6.1; no longer C5.1
- net N$3: now also C5.1; no longer C4.1
- net N$5: now also C4.1; no longer C3.1
- net N$6: now also C12.1; no longer C11.1
- net PREVGH: now also C11.1; no longer C10.1
- net PREVGL: now also C13.1; no longer C12.1
Routing:
- net +3V3: track 91.0 -> 113.4 mm
- net N$4: track 12.8 -> 0.00 mm
- net 0V: track 59.4 -> 62.1 mm
