File: epaper_eval/WFT0750CZ09_conv.sch (EAGLE design)
At the start: 26 parts, among them CN1 WFT0750CZ09_IF, CN2 WFT0750CZ09-SMD_, Q1 PMF370XN_, U1 LM75BIMM-3_

Commit message: 基板デザイン修正
Parts:
- C7: device Parts:TPST106K016R0800 -> Parts:TPST106K016R0800_
- L1: device Parts:NLCV25T -> Parts:NLCV25T_
Changed lines of the file:
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@@
 <part name="GND1" library="Supply" deviceset="0V" device=""/>
 <part name="C9" library="Parts" deviceset="CAP" device="_0805" value="0.1uF16V"/>
-<part name="L1" library="Parts" deviceset="NLCV*" device="25T" value="10uH"/>
+<part name="L1" library="Parts" deviceset="NLCV*" device="25T_" value="10uH"/>
 <part name="Q1" library="Parts" deviceset="PMF370XN" device="_"/>
 <part name="R3" library="Parts" deviceset="RESISTOR" device="_0805" value="0.47"/>
@@
 <part name="C13" library="Parts" deviceset="CAP" device="_0805" value="0.1uF50V"/>
 <part name="R2" library="Parts" deviceset="RESISTOR" device="_0805" value="100k"/>
-<part name="C7" library="Parts" deviceset="TPST*" device="106K016R0800" value="10uF16V"/>
+<part name="C7" library="Parts" deviceset="TPST*" device="106K016R0800_" value="10uF16V"/>
 <part name="R1" library="Parts" deviceset="RESISTOR" device="_0805" value="10"/>
 <part name="C8" library="Parts" deviceset="CAP" device="_0805" value="1uF16V"/>

Commit message: 部品変更
Parts:
- removed R1: 10, Parts:RESISTOR_0805
- added C14: 0.1uF50V, Parts:CAP_0805
- C10: value 10uF50V -> 0.1uF16V
- C11: value 4.7uF50V -> 10uF50V
- C12: value 10uF50V -> 4.7uF50V
- C13: value 0.1uF50V -> 10uF50V
- C4: value 10uF50V -> 1uF50V
- C6: value 1uF50V -> 10uF50V
- C7: value 10uF16V -> 1uF50V; device Parts:TPST106K016R0800_ -> Parts:CAP_0805
- C8: value 1uF16V -> 10uF16V; device Parts:CAP_0805 -> Parts:TPST106K016R0800_
- C9: value 0.1uF16V -> 1uF16V
Connections:
- removed net N$4: CN2.VCI, CN2.VDDIO, R1.2
- net +3V3: now also C10.1, C14.1, C3.1, C8.+, CN2.VCI, CN2.VDDIO; no longer C13.1, C7.+, C8.1, R1.1
- net 0V: now also C11.2, C14.2, C7.2, C8.-; no longer C12.2, C7.-, C8.2
- net N$1: now also C7.1; no longer C6.1
- net N$15: now also C12.2; no longer C11.2
- net N$2: now also C6.1; no longer C5.1
- net N$3: now also C5.1; no longer C4.1
- net N$5: now also C4.1; no longer C3.1
- net N$6: now also C12.1; no longer C11.1
- net PREVGH: now also C11.1; no longer C10.1
- net PREVGL: now also C13.1; no longer C12.1
Other:
- moved on the sheet: C1, C10, C11, C12, C13, C2, C3, C4, C5, C6, C9
